File: USB_POWER.kicad_sch (KiCad schematic)
At the start: 26 parts, among them J601 TYPE-C-32-M-12, U601 LN1134A332MR-G, U602 C5451661, U603 C5451661, U604 74LVC1G08, U605 BL1551B, U606 BL1551B, U607 BL1551B, U608 BL1551B

Commit message: Updates F.Silkscreen
Parts:
- J601: footprint suku_basics:USB_C_Korean_Hroparts_TYPE-C-31-M-12 -> Connector_USB:USB_C_Receptacle_GCT_USB4105-xx-A_16P_TopMnt_Horizontal
Changed lines of the file:
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@@
 			)
 		)
-		(property "Footprint" "suku_basics:USB_C_Korean_Hroparts_TYPE-C-31-M-12"
+		(property "Footprint" "Connector_USB:USB_C_Receptacle_GCT_USB4105-xx-A_16P_TopMnt_Horizontal"
 			(at 40.64 73.66 0)
 			(effects
